File: RDB_STPTS_002.kicad_pcb (KiCad board)
At the start: 2 copper layers, 159.4 x 99.7 mm, 240 parts

Commit message: cleanup
Other:
- board text removed: "resistori pt leduri 12-40v la 2k2 ?? adaugat led pt pswitch power in la capat siguranta de 6,3mm nu se potriveste resistori serie protectie linii digital 270-1k ??? feturi cu leduri pt stare endstopuri???"
Changed lines of the file:
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@@
     (links 499)
     (no_connects 0)
-    (area 31.207529 23.82 210.565 144.43)
+    (area 31.207529 23.82 210.565 140.83)
     (thickness 1.6)
-    (drawings 31)
+    (drawings 30)
     (tracks 1461)
     (zones 0)
@@
     )
   )
-  (gr_text "resistori pt leduri 12-40v la 2k2 ??\nadaugat led pt pswitch power in la capat\nsiguranta de 6,3mm nu se potriveste\nresistori serie protectie linii digital 270-1k ???\nfeturi cu leduri pt stare endstopuri???" (at 108.585 138.43) (layer F.Cu)
-    (effects (font (size 1.5 1.5) (thickness 0.3)))
-  )
   (gr_line (start 162.56 77.47) (end 185.1025 77.47) (angle 90) (layer Edge.Cuts) (width 0.1))
